File: AirlabMuxAtmel.kicad_pcb (KiCad board)
At the start: 2 copper layers, 2 parts, among them IC1 ATXMEGA128A4U#TQFP44, IC2 80C552

Commit message: ok
ok
Connections:
- IC1 pad 1: LCD_RS -> LCD_E
- IC1 pad 2: LCD_E -> LCD_RS
- IC1 pad 43: LCD_D7 -> LCD_RW
- IC1 pad 44: LCD_RW -> LCD_D7
Routing:
- net LCD_D6: track 0.00 -> 12.3 mm
- net LCD_D4: track 0.00 -> 11.2 mm
- net LCD_D7: track 0.00 -> 10.3 mm
- net LCD_RW: track 0.00 -> 9.13 mm
- net LCD_RS: track 0.00 -> 8.57 mm
- net LCD_D5: track 0.00 -> 8.25 mm
- net LCD_E: track 0.00 -> 5.70 mm
Changed lines of the file:
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@@
     (fp_line (start 5 5) (end -5 5) (layer "F.Fab") (width 0.15))
     (pad "1" smd rect locked (at -5.7 -4) (size 1.5 0.55) (layers "F.Cu" "F.Paste" "F.Mask")
-      (net 1 "LCD_RS") (pinfunction "AC5/ADC5/PA5") (pintype "bidirectional"))
+      (net 36 "LCD_E") (pinfunction "AC5/ADC5/PA5") (pintype "bidirectional"))
     (pad "2" smd rect locked (at -5.7 -3.2) (size 1.5 0.55) (layers "F.Cu" "F.Paste" "F.Mask")
-      (net 36 "LCD_E") (pinfunction "AC1OUT/AC6/ADC6/PA6") (pintype "bidirectional"))
+      (net 1 "LCD_RS") (pinfunction "AC1OUT/AC6/ADC6/PA6") (pintype "bidirectional"))
     (pad "3" smd rect locked (at -5.7 -2.4) (size 1.5 0.55) (layers "F.Cu" "F.Paste" "F.Mask")
       (net 2 "unconnected-(IC1-Pad3)") (pinfunction "AC0OUT/AC7/ADC7/PA7") (pintype "bidirectional"))
@@
       (net 39 "LCD_D6") (pinfunction "AC2/ADC2/PA2") (pintype "bidirectional"))
     (pad "43" smd rect locked (at -3.2 -5.7 90) (size 1.5 0.55) (layers "F.Cu" "F.Paste" "F.Mask")
-      (net 45 "LCD_D7") (pinfunction "AC3/ADC3/PA3") (pintype "bidirectional"))
+      (net 46 "LCD_RW") (pinfunction "AC3/ADC3/PA3") (pintype "bidirectional"))
     (pad "44" smd rect locked (at -4 -5.7 90) (size 1.5 0.55) (layers "F.Cu" "F.Paste" "F.Mask")
-      (net 46 "LCD_RW") (pinfunction "AC4/ADC4/PA4") (pintype "bidirectional"))
+      (net 45 "LCD_D7") (pinfunction "AC4/ADC4/PA4") (pintype "bidirectional"))
     (model "${KISYS3DMOD}/TQFP-44_10x10mm_P0.8mm.step"
       (offset (xyz 0 0 0))
@@
     )
   )
+  (segment (start 88.264282 60.325) (end 86.36 60.325) (width 0.25) (layer "F.Cu") (net 1))
+  (segment (start 86.36 60.325) (end 85.09 59.055) (width 0.25) (layer "F.Cu") (net 1))
+  (segment (start 92.09 62.84) (end 90.779282 62.84) (width 0.25) (layer "F.Cu") (net 1))
+  (segment (start 90.779282 62.84) (end 88.264282 60.325) (width 0.25) (layer "F.Cu") (net 1))
+  (segment (start 90.615 62.04) (end 87.63 59.055) (width 0.25) (layer "F.Cu") (net 36))
+  (segment (start 92.09 62.04) (end 90.615 62.04) (width 0.25) (layer "F.Cu") (net 36))
+  (segment (start 92.202 57.912) (end 91.44 57.15) (width 0.25) (layer "F.Cu") (net 37))
+  (segment (start 91.44 57.15) (end 91.44 55.245) (width 0.25) (layer "F.Cu") (net 37))
+  (segment (start 91.44 55.245) (end 90.17 53.975) (width 0.25) (layer "F.Cu") (net 37))
+  (segment (start 96.99 60.34) (end 96.99 59.271) (width 0.25) (layer "F.Cu") (net 37))
+  (segment (start 96.99 59.271) (end 95.631 57.912) (width 0.25) (layer "F.Cu") (net 37))
+  (segment (start 95.631 57.912) (end 92.202 57.912) (width 0.25) (layer "F.Cu") (net 37))
+  (segment (start 95.31852 58.36152) (end 92.015802 58.36152) (width 0.25) (layer "F.Cu") (net 38))
+  (segment (start 90.17 56.515718) (end 90.17 56.515) (width 0.25) (layer "F.Cu") (net 38))
+  (segment (start 96.19 60.34) (end 96.19 59.233) (width 0.25) (layer "F.Cu") (net 38))
+  (segment (start 92.015802 58.36152) (end 90.17 56.515718) (width 0.25) (layer "F.Cu") (net 38))
+  (segment (start 96.19 59.233) (end 95.31852 58.36152) (width 0.25) (layer "F.Cu") (net 38))
+  (segment (start 91.70404 58.81104) (end 90.73648 57.84348) (width 0.25) (layer "F.Cu") (net 39))
+  (segment (start 88.9 55.6895) (end 87.63 54.4195) (width 0.25) (layer "F.Cu") (net 39))
+  (segment (start 90.73648 57.84348) (end 89.594198 57.84348) (width 0.25) (layer "F.Cu") (net 39))
+  (segment (start 95.39 60.34) (end 95.39 59.068718) (width 0.25) (layer "F.Cu") (net 39))
+  (segment (start 95.132322 58.81104) (end 91.70404 58.81104) (width 0.25) (layer "F.Cu") (net 39))
+  (segment (start 87.63 54.4195) (end 87.63 53.975) (width 0.25) (layer "F.Cu") (net 39))
+  (segment (start 95.39 59.068718) (end 95.132322 58.81104) (width 0.25) (layer "F.Cu") (net 39))
+  (segment (start 88.9 57.149282) (end 88.9 55.6895) (width 0.25) (layer "F.Cu") (net 39))
+  (segment (start 89.594198 57.84348) (end 88.9 57.149282) (width 0.25) (layer "F.Cu") (net 39))
+  (segment (start 90.693 60.34) (end 88.138 57.785) (width 0.25) (layer "F.Cu") (net 45))
+  (segment (start 93.79 60.34) (end 90.693 60.34) (width 0.25) (layer "F.Cu") (net 45))
+  (segment (start 88.138 57.785) (end 86.36 57.785) (width 0.25) (layer "F.Cu") (net 45))
+  (segment (start 86.36 57.785) (end 85.09 56.515) (width 0.25) (layer "F.Cu") (net 45))
+  (segment (start 87.63 56.515) (end 89.408 58.293) (width 0.25) (layer "F.Cu") (net 46))
+  (segment (start 94.59 59.34) (end 94.59 60.34) (width 0.25) (layer "F.Cu") (net 46))
+  (segment (start 91.517842 59.26056) (end 94.51056 59.26056) (width 0.25) (layer "F.Cu") (net 46))
+  (segment (start 94.51056 59.26056) (end 94.59 59.34) (width 0.25) (layer "F.Cu") (net 46))
+  (segment (start 89.408 58.293) (end 90.550282 58.293) (width 0.25) (layer "F.Cu") (net 46))
+  (segment (start 90.550282 58.293) (end 91.517842 59.26056) (width 0.25) (layer "F.Cu") (net 46))
 )

Commit message: oke
oke
Parts:
- added C2: 100N-X7R_50V#0603-D&R_Passive, D&R_Passive:C_0603, F.Cu at (99.3, 74.4)
- added C3: 100N-X7R_50V#0603-D&R_Passive, D&R_Passive:C_0603, F.Cu at (97.8, 57.9)
- added IC3: ATXMEGA128A4U#TQFP44, Package_qfn:QFN50P700X700X100-45N, F.Cu at (97.8, 66.0)
- added P1: CONN_02X03, D&R_Conn:HEADER_2x3P, F.Cu at (109.2, 64.1)
- added R1: 0R#0603, D&R_Passive:R_0603, F.Cu at (110.7, 54.1)
Connections:
- IC1 pad 10: unconnected-(IC1-Pad10) -> AS2
- IC1 pad 11: unconnected-(IC1-Pad11) -> STRB2
- IC1 pad 12: unconnected-(IC1-Pad12) -> AS4
- IC1 pad 13: unconnected-(IC1-Pad13) -> DATA1
- IC1 pad 14: unconnected-(IC1-Pad14) -> CLK1
- IC1 pad 15: unconnected-(IC1-Pad15) -> DATA2
- IC1 pad 16: unconnected-(IC1-Pad16) -> CLK2
- IC1 pad 17: unconnected-(IC1-Pad17) -> CS_CC
- IC1 pad 19: unconnected-(IC1-Pad19) -> Net-(C2-Pad1)
- IC1 pad 22: unconnected-(IC1-Pad22) -> SW4
- IC1 pad 23: unconnected-(IC1-Pad23) -> SW3
- IC1 pad 24: unconnected-(IC1-Pad24) -> SW8
- IC1 pad 25: unconnected-(IC1-Pad25) -> SW7
- IC1 pad 26: unconnected-(IC1-Pad26) -> SW6
- IC1 pad 27: unconnected-(IC1-Pad27) -> SW5
- IC1 pad 28: unconnected-(IC1-Pad28) -> SDA
- IC1 pad 29: unconnected-(IC1-Pad29) -> SCL
- IC1 pad 3: unconnected-(IC1-Pad3) -> RST_CC
- IC1 pad 31: unconnected-(IC1-Pad31) -> Net-(C2-Pad1)
- IC1 pad 32: unconnected-(IC1-Pad32) -> RXD
- IC1 pad 33: unconnected-(IC1-Pad33) -> TXD
- IC1 pad 34: unconnected-(IC1-Pad34) -> Net-(IC1-Pad34)
- IC1 pad 35: unconnected-(IC1-Pad35) -> Net-(IC1-Pad35)
- IC1 pad 36: unconnected-(IC1-Pad36) -> SW2
- IC1 pad 37: unconnected-(IC1-Pad37) -> SW1
- IC1 pad 39: unconnected-(IC1-Pad39) -> Net-(C2-Pad1)
- IC1 pad 4: unconnected-(IC1-Pad4) -> STRB1
- IC1 pad 5: unconnected-(IC1-Pad5) -> AS1
- IC1 pad 6: unconnected-(IC1-Pad6) -> AS0
- IC1 pad 7: unconnected-(IC1-Pad7) -> AS3
- IC1 pad 9: unconnected-(IC1-Pad9) -> Net-(C2-Pad1)
- IC2 pad 1: unconnected-(IC2-Pad1) -> SW1
- IC2 pad 14: unconnected-(IC2-Pad14) -> STRB1
- IC2 pad 16: unconnected-(IC2-Pad16) -> AS0
- IC2 pad 17: unconnected-(IC2-Pad17) -> AS1
- IC2 pad 18: unconnected-(IC2-Pad18) -> AS2
- IC2 pad 19: unconnected-(IC2-Pad19) -> AS3
- IC2 pad 2: unconnected-(IC2-Pad2) -> Net-(C2-Pad1)
- IC2 pad 20: unconnected-(IC2-Pad20) -> AS4
- IC2 pad 21: unconnected-(IC2-Pad21) -> STRB2
- IC2 pad 22: unconnected-(IC2-Pad22) -> SCL
- IC2 pad 23: unconnected-(IC2-Pad23) -> SDA
- IC2 pad 24: unconnected-(IC2-Pad24) -> RXD
- IC2 pad 25: unconnected-(IC2-Pad25) -> TXD
- IC2 pad 26: unconnected-(IC2-Pad26) -> DATA1
- IC2 pad 27: unconnected-(IC2-Pad27) -> DATA2
- IC2 pad 28: unconnected-(IC2-Pad28) -> CLK1
- IC2 pad 29: unconnected-(IC2-Pad29) -> CLK2
- IC2 pad 4: unconnected-(IC2-Pad4) -> RST_CC
- IC2 pad 5: unconnected-(IC2-Pad5) -> CS_CC
- IC2 pad 62: unconnected-(IC2-Pad62) -> SW8
- IC2 pad 63: unconnected-(IC2-Pad63) -> SW7
- IC2 pad 64: unconnected-(IC2-Pad64) -> SW6
- IC2 pad 65: unconnected-(IC2-Pad65) -> SW5
- IC2 pad 66: unconnected-(IC2-Pad66) -> SW4
- IC2 pad 67: unconnected-(IC2-Pad67) -> SW3
- IC2 pad 68: unconnected-(IC2-Pad68) -> SW2
Routing:
- net Net-(C2-Pad1): track 0.00 -> 100.0 mm, vias 0 -> 3
- net Net-(C2-Pad2): track 0.00 -> 57.3 mm, vias 0 -> 17
- net RXD: track 0.00 -> 50.7 mm, vias 0 -> 1
- net CS_CC: track 0.00 -> 42.9 mm, vias 0 -> 1
- net SCL: track 0.00 -> 40.3 mm, vias 0 -> 2
- net SDA: track 0.00 -> 37.5 mm, vias 0 -> 2
- net TXD: track 0.00 -> 35.9 mm, vias 0 -> 2
- net SW4: track 0.00 -> 29.4 mm, vias 0 -> 1
- net Net-(IC1-Pad35): track 0.00 -> 27.1 mm, vias 0 -> 2
- net SW3: track 0.00 -> 24.0 mm, vias 0 -> 1
- net SW7: track 0.00 -> 20.0 mm
- net SW8: track 0.00 -> 18.4 mm
- net SW5: track 0.00 -> 17.8 mm
- net DATA2: track 0.00 -> 16.6 mm
- net RST_CC: track 0.00 -> 16.5 mm, vias 0 -> 1
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- added copper zone on B.Cu, net Net-(C2-Pad2)
- added copper zone on F.Cu, net Net-(C2-Pad2)
Other:
- board outline added: 32 x 32 mm
